Commit message: feat: Refactor joint configuration and improve inference thread handling for Muto robot

File: muto_ws/src/muto_description/urdf/Muto_complet.urdf.xacro (robot description, xacro)
@@ -17,4 +17,71 @@
       <param name="torque_enabled">true</param>
     </hardware>
+    <!-- ─── RIGHT SIDE ────────────────────────────────────────── -->
+    <!-- yq - Front Right -->
+    <joint name="yq1_Joint">
+      <command_interface name="position">
+        <param name="min">-1.2</param>
+        <param name="max">1.2</param>
+      </command_interface>
+      <state_interface name="position"/>
+    </joint>
+    <joint name="yq2_Joint">
+      <command_interface name="position">
+        <param name="min">-1.57</param>
+        <param name="max">1.57</param>
+      </command_interface>
+      <state_interface name="position"/>
+    </joint>
+    <joint name="yq3_Joint">
+      <command_interface name="position">
+        <param name="min">-1.57</param>
+        <param name="max">0.7</param>
+      </command_interface>
+      <state_interface name="position"/>
+    </joint>
+    <!-- yz - Mid Right -->
+    <joint name="yz1_Joint">
+      <command_interface name="position">
+        <param name="min">-1.2</param>
+        <param name="max">1.2</param>
+      </command_interface>
+      <state_interface name="position"/>
+    </joint>
+    <joint name="yz2_Joint">
+      <command_interface name="position">
+        <param name="min">-1.57</param>
+        <param name="max">1.57</param>
+      </command_interface>
+      <state_interface name="position"/>
+    </joint>
+    <joint name="yz3_Joint">
+      <command_interface name="position">
+        <param name="min">-1.57</param>
+        <param name="max">0.7</param>
+      </command_interface>
+      <state_interface name="position"/>
+    </joint>
+    <!-- yh - Rear Right -->
+    <joint name="yh1_Joint">
+      <command_interface name="position">
+        <param name="min">-1.2</param>
+        <param name="max">1.2</param>
+      </command_interface>
+      <state_interface name="position"/>
+    </joint>
+    <joint name="yh2_Joint">
+      <command_interface name="position">
+        <param name="min">-1.57</param>
+        <param name="max">1.57</param>
+      </command_interface>
+      <state_interface name="position"/>
+    </joint>
+    <joint name="yh3_Joint">
+      <command_interface name="position">
+        <param name="min">-1.57</param>
+        <param name="max">0.7</param>
+      </command_interface>
+      <state_interface name="position"/>
+    </joint>
     <!-- ─── LEFT SIDE ─────────────────────────────────────────── -->
     <!-- zq - Front Left -->
@@ -84,71 +151,4 @@
       <state_interface name="position"/>
     </joint>
-    <!-- ─── RIGHT SIDE ────────────────────────────────────────── -->
-    <!-- yq - Front Right -->
-    <joint name="yq1_Joint">
-      <command_interface name="position">
-        <param name="min">-1.2</param>
-        <param name="max">1.2</param>
-      </command_interface>
-      <state_interface name="position"/>
-    </joint>
-    <joint name="yq2_Joint">
-      <command_interface name="position">
-        <param name="min">-1.57</param>
-        <param name="max">1.57</param>
-      </command_interface>
-      <state_interface name="position"/>
-    </joint>
-    <joint name="yq3_Joint">
-      <command_interface name="position">
-        <param name="min">-1.57</param>
-        <param name="max">0.7</param>
-      </command_interface>
-      <state_interface name="position"/>
-    </joint>
-    <!-- yz - Mid Right -->
-    <joint name="yz1_Joint">
-      <command_interface name="position">
-        <param name="min">-1.2</param>
-        <param name="max">1.2</param>
-      </command_interface>
-      <state_interface name="position"/>
-    </joint>
-    <joint name="yz2_Joint">
-      <command_interface name="position">
-        <param name="min">-1.57</param>
-        <param name="max">1.57</param>
-      </command_interface>
-      <state_interface name="position"/>
-    </joint>
-    <joint name="yz3_Joint">
-      <command_interface name="position">
-        <param name="min">-1.57</param>
-        <param name="max">0.7</param>
-      </command_interface>
-      <state_interface name="position"/>
-    </joint>
-    <!-- yh - Rear Right -->
-    <joint name="yh1_Joint">
-      <command_interface name="position">
-        <param name="min">-1.2</param>
-        <param name="max">1.2</param>
-      </command_interface>
-      <state_interface name="position"/>
-    </joint>
-    <joint name="yh2_Joint">
-      <command_interface name="position">
-        <param name="min">-1.57</param>
-        <param name="max">1.57</param>
-      </command_interface>
-      <state_interface name="position"/>
-    </joint>
-    <joint name="yh3_Joint">
-      <command_interface name="position">
-        <param name="min">-1.57</param>
-        <param name="max">0.7</param>
-      </command_interface>
-      <state_interface name="position"/>
-    </joint>
   </ros2_control>
 </robot>

File: muto_ws/src/muto_description/urdf/Muto_gazebo.urdf.xacro (robot description, xacro)
@@ -12,4 +12,44 @@
       <plugin>gz_ros2_control/GazeboSimSystem</plugin>
     </hardware>
+    <!-- ─── RIGHT SIDE ────────────────────────────────────────── -->
+    <!-- yq - Front Right -->
+    <joint name="yq1_Joint">
+      <command_interface name="position"><param name="min">-1.2</param><param name="max">1.2</param></command_interface>
+      <state_interface name="position"/>
+    </joint>
+    <joint name="yq2_Joint">
+      <command_interface name="position"><param name="min">-1.57</param><param name="max">1.57</param></command_interface>
+      <state_interface name="position"/>
+    </joint>
+    <joint name="yq3_Joint">
+      <command_interface name="position"><param name="min">-1.57</param><param name="max">0.7</param></command_interface>
+      <state_interface name="position"/>
+    </joint>
+    <!-- yz - Mid Right -->
+    <joint name="yz1_Joint">
+      <command_interface name="position"><param name="min">-1.2</param><param name="max">1.2</param></command_interface>
+      <state_interface name="position"/>
+    </joint>
+    <joint name="yz2_Joint">
+      <command_interface name="position"><param name="min">-1.57</param><param name="max">1.57</param></command_interface>
+      <state_interface name="position"/>
+    </joint>
+    <joint name="yz3_Joint">
+      <command_interface name="position"><param name="min">-1.57</param><param name="max">0.7</param></command_interface>
+      <state_interface name="position"/>
+    </joint>
+    <!-- yh - Rear Right -->
+    <joint name="yh1_Joint">
+      <command_interface name="position"><param name="min">-1.2</param><param name="max">1.2</param></command_interface>
+      <state_interface name="position"/>
+    </joint>
+    <joint name="yh2_Joint">
+      <command_interface name="position"><param name="min">-1.57</param><param name="max">1.57</param></command_interface>
+      <state_interface name="position"/>
+    </joint>
+    <joint name="yh3_Joint">
+      <command_interface name="position"><param name="min">-1.57</param><param name="max">0.7</param></command_interface>
+      <state_interface name="position"/>
+    </joint>
     <!-- ─── LEFT SIDE ─────────────────────────────────────────── -->
     <!-- zq - Front Left -->
@@ -52,44 +92,4 @@
       <state_interface name="position"/>
     </joint>
-    <!-- ─── RIGHT SIDE ────────────────────────────────────────── -->
-    <!-- yq - Front Right -->
-    <joint name="yq1_Joint">
-      <command_interface name="position"><param name="min">-1.2</param><param name="max">1.2</param></command_interface>
-      <state_interface name="position"/>
-    </joint>
-    <joint name="yq2_Joint">
-      <command_interface name="position"><param name="min">-1.57</param><param name="max">1.57</param></command_interface>
-      <state_interface name="position"/>
-    </joint>
-    <joint name="yq3_Joint">
-      <command_interface name="position"><param name="min">-1.57</param><param name="max">0.7</param></command_interface>
-      <state_interface name="position"/>
-    </joint>
-    <!-- yz - Mid Right -->
-    <joint name="yz1_Joint">
-      <command_interface name="position"><param name="min">-1.2</param><param name="max">1.2</param></command_interface>
-      <state_interface name="position"/>
-    </joint>
-    <joint name="yz2_Joint">
-      <command_interface name="position"><param name="min">-1.57</param><param name="max">1.57</param></command_interface>
-      <state_interface name="position"/>
-    </joint>
-    <joint name="yz3_Joint">
-      <command_interface name="position"><param name="min">-1.57</param><param name="max">0.7</param></command_interface>
-      <state_interface name="position"/>
-    </joint>
-    <!-- yh - Rear Right -->
-    <joint name="yh1_Joint">
-      <command_interface name="position"><param name="min">-1.2</param><param name="max">1.2</param></command_interface>
-      <state_interface name="position"/>
-    </joint>
-    <joint name="yh2_Joint">
-      <command_interface name="position"><param name="min">-1.57</param><param name="max">1.57</param></command_interface>
-      <state_interface name="position"/>
-    </joint>
-    <joint name="yh3_Joint">
-      <command_interface name="position"><param name="min">-1.57</param><param name="max">0.7</param></command_interface>
-      <state_interface name="position"/>
-    </joint>
   </ros2_control>
   <!-- Plugin required to connect ros2_control to Gazebo -->
