Commit message: Add ROS 2 control configuration and launch files for MUTO-RS hexapod
- Updated Muto_complet.urdf.xacro to include hardware interface parameters and joint limits for 18 joints.
- Created controllers.yaml to define the controller manager and leg controller parameters.
- Added bringup.launch.py to launch the robot state publisher and controller manager with spawners for joint state broadcaster and leg controller.
- Introduced muto_hardware_plugin.xml to define the hardware interface plugin for the MUTO-RS hexapod.

File: muto_ws/src/muto_description/urdf/Muto.urdf (robot description, URDF)
Before this commit: robot yahboomcar, 24 links, 23 joints
Joints:
- removed joint yh2_Link
- removed joint yh3_Link
- added joint yh2_Joint: type revolute, parent yh1_Link, child yh2_Link, origin xyz=-0.055226635669978 -0.0165734288280502 -0.027473927115545 rpy=0 0 0, axis -0.711636313809332 0.702548045949788 0, limit lower=-1.57 upper=1.57 effort=2.5 velocity=3.14
- added joint yh3_Joint: type revolute, parent yh2_Link, child yh3_Link, origin xyz=-0.0497740601308654 -0.0504179449064808 0.0158615312365509 rpy=0 0 0, axis 0.711636313809335 -0.702548045949785 0, limit lower=-1.57 upper=1.57 effort=2.5 velocity=3.14
- joint yh1_Joint: limit lower=-1.57 upper=1.57 effort=0 velocity=0 -> lower=-1.57 upper=1.57 effort=2.5 velocity=3.14
- joint yq1_Joint: limit lower=-1.57 upper=1.57 effort=0 velocity=0 -> lower=-1.57 upper=1.57 effort=2.5 velocity=3.14
- joint yq2_Joint: limit lower=-1.57 upper=1.57 effort=0 velocity=0 -> lower=-1.57 upper=1.57 effort=2.5 velocity=3.14
- joint yq3_Joint: limit lower=-1.57 upper=1.57 effort=0 velocity=0 -> lower=-1.57 upper=1.57 effort=2.5 velocity=3.14
- joint yz1_Joint: limit lower=-1.57 upper=1.57 effort=0 velocity=0 -> lower=-1.57 upper=1.57 effort=2.5 velocity=3.14
- joint yz2_Joint: limit lower=-1.57 upper=1.57 effort=0 velocity=0 -> lower=-1.57 upper=1.57 effort=2.5 velocity=3.14
- joint yz3_Joint: limit lower=-1.57 upper=1.57 effort=0 velocity=0 -> lower=-1.57 upper=1.57 effort=2.5 velocity=3.14
- joint zh1_Joint: limit lower=-1.57 upper=1.57 effort=0 velocity=0 -> lower=-1.57 upper=1.57 effort=2.5 velocity=3.14
- joint zh2_Joint: limit lower=-1.57 upper=1.57 effort=0 velocity=0 -> lower=-1.57 upper=1.57 effort=2.5 velocity=3.14
- joint zh3_Joint: limit lower=-1.57 upper=1.57 effort=0 velocity=0 -> lower=-1.57 upper=1.57 effort=2.5 velocity=3.14
- joint zq1_Joint: limit lower=-1.57 upper=1.57 effort=0 velocity=0 -> lower=-1.57 upper=1.57 effort=2.5 velocity=3.14
- joint zq2_Joint: limit lower=-1.57 upper=1.57 effort=0 velocity=0 -> lower=-1.57 upper=1.57 effort=2.5 velocity=3.14
- joint zq3_Joint: limit lower=-1.57 upper=1.57 effort=0 velocity=0 -> lower=-1.57 upper=1.57 effort=2.5 velocity=3.14
- joint zz1_Joint: limit lower=-1.57 upper=1.57 effort=0 velocity=0 -> lower=-1.57 upper=1.57 effort=2.5 velocity=3.14
- joint zz2_Joint: limit lower=-1.57 upper=1.57 effort=0 velocity=0 -> lower=-1.57 upper=1.57 effort=2.5 velocity=3.14
- joint zz3_Joint: limit lower=-1.57 upper=1.57 effort=0 velocity=0 -> lower=-1.57 upper=1.57 effort=2.5 velocity=3.14

File: muto_ws/src/muto_description/urdf/Muto_complet.urdf.xacro (robot description, xacro)
@@ -1,90 +1,148 @@
 <?xml version="1.0"?>
-<robot xmlns:xacro="http://ros.org" name="muto_robot">
-    <!-- 1. Inclure votre fichier URDF original -->
-    <xacro:include filename="Muto.urdf" />
-    <!-- 2. Ajouter la configuration ros2_control par-dessus -->
-    <ros2_control name="MutoHardwareInterface" type="system">
-        <hardware>
-            <plugin>topic_based_ros2_control/TopicBasedSystemInterface</plugin>
-        </hardware>
-        <!-- Déclaration de vos 18 articulations -->
-        <!-- zq -->
-        <joint name="zq1_Joint">
-            <command_interface name="position"/>
-            <state_interface name="position"/>
-        </joint>
-        <joint name="zq2_Joint">
-            <command_interface name="position"/>
-            <state_interface name="position"/>
-        </joint>
-        <joint name="zq3_Joint">
-            <command_interface name="position"/>
-            <state_interface name="position"/>
-        </joint>
-        <!-- zz -->
-        <joint name="zz1_Joint">
-            <command_interface name="position"/>
-            <state_interface name="position"/>
-        </joint>
-        <joint name="zz2_Joint">
-            <command_interface name="position"/>
-            <state_interface name="position"/>
-        </joint>
-        <joint name="zz3_Joint">
-            <command_interface name="position"/>
-            <state_interface name="position"/>
-        </joint>
-        <!-- zh -->
-        <joint name="zh1_Joint">
-            <command_interface name="position"/>
-            <state_interface name="position"/>
-        </joint>
-        <joint name="zh2_Joint">
-            <command_interface name="position"/>
-            <state_interface name="position"/>
-        </joint>
-        <joint name="zh3_Joint">
-            <command_interface name="position"/>
-            <state_interface name="position"/>
-        </joint>
-        <!-- yq -->
-        <joint name="yq1_Joint">
-            <command_interface name="position"/>
-            <state_interface name="position"/>
-        </joint>
-        <joint name="yq2_Joint">
-            <command_interface name="position"/>
-            <state_interface name="position"/>
-        </joint>
-        <joint name="yq3_Joint">
-            <command_interface name="position"/>
-            <state_interface name="position"/>
-        </joint>
-        <!-- yz -->
-        <joint name="yz1_Joint">
-            <command_interface name="position"/>
-            <state_interface name="position"/>
-        </joint>
-        <joint name="yz2_Joint">
-            <command_interface name="position"/>
-            <state_interface name="position"/>
-        </joint>
-        <joint name="yz3_Joint">
-            <command_interface name="position"/>
-            <state_interface name="position"/>
-        </joint>
-        <!-- yh -->
-        <joint name="yh1_Joint">
-            <command_interface name="position"/>
-            <state_interface name="position"/>
-        </joint>
-        <joint name="yh2_Joint">
-            <command_interface name="position"/>
-            <state_interface name="position"/>
-        </joint>
-        <joint name="yh3_Joint">
-            <command_interface name="position"/>
-            <state_interface name="position"/>
-        </joint>
-    </ros2_control>
+<robot xmlns:xacro="http://www.ros.org/wiki/xacro" name="muto_robot">
+  <xacro:include filename="$(find muto_description)/urdf/Muto.urdf"/>
+  <ros2_control name="MutoHardwareInterface" type="system">
+    <hardware>
+      <plugin>muto_hardware/MutoHexapodHardware</plugin>
+      <param name="port">/dev/ttyUSB0</param>
+      <param name="baud">115200</param>
+      <param name="read_timeout_sec">0.05</param>
+      <param name="retry_count">2</param>
+      <param name="validate_checksum">true</param>
+      <param name="servo_speed">300</param>
+      <param name="servo_ids">1 2 3 4 5 6 7 8 9 10 11 12 13 14 15 16 17 18</param>
+    </hardware>
+    <!-- zq - front right -->
+    <joint name="zq1_Joint">
+      <command_interface name="position">
+        <param name="min">-1.57</param>
+        <param name="max">1.57</param>
+      </command_interface>
+      <state_interface name="position"/>
+    </joint>
+    <joint name="zq2_Joint">
+      <command_interface name="position">
+        <param name="min">-1.57</param>
+        <param name="max">1.57</param>
+      </command_interface>
+      <state_interface name="position"/>
+    </joint>
+    <joint name="zq3_Joint">
+      <command_interface name="position">
+        <param name="min">-1.57</param>
+        <param name="max">1.57</param>
+      </command_interface>
+      <state_interface name="position"/>
+    </joint>
+    <!-- zz - mid right -->
+    <joint name="zz1_Joint">
+      <command_interface name="position">
+        <param name="min">-1.57</param>
+        <param name="max">1.57</param>
+      </command_interface>
+      <state_interface name="position"/>
+    </joint>
+    <joint name="zz2_Joint">
+      <command_interface name="position">
+        <param name="min">-1.57</param>
+        <param name="max">1.57</param>
+      </command_interface>
+      <state_interface name="position"/>
+    </joint>
+    <joint name="zz3_Joint">
+      <command_interface name="position">
+        <param name="min">-1.57</param>
+        <param name="max">1.57</param>
+      </command_interface>
+      <state_interface name="position"/>
+    </joint>
+    <!-- zh - rear right -->
+    <joint name="zh1_Joint">
+      <command_interface name="position">
+        <param name="min">-1.57</param>
+        <param name="max">1.57</param>
+      </command_interface>
+      <state_interface name="position"/>
+    </joint>
+    <joint name="zh2_Joint">
+      <command_interface name="position">
+        <param name="min">-1.57</param>
+        <param name="max">1.57</param>
+      </command_interface>
+      <state_interface name="position"/>
+    </joint>
+    <joint name="zh3_Joint">
+      <command_interface name="position">
+        <param name="min">-1.57</param>
+        <param name="max">1.57</param>
+      </command_interface>
+      <state_interface name="position"/>
+    </joint>
+    <!-- yq - front left -->
+    <joint name="yq1_Joint">
+      <command_interface name="position">
+        <param name="min">-1.57</param>
+        <param name="max">1.57</param>
+      </command_interface>
+      <state_interface name="position"/>
+    </joint>
+    <joint name="yq2_Joint">
+      <command_interface name="position">
+        <param name="min">-1.57</param>
+        <param name="max">1.57</param>
+      </command_interface>
+      <state_interface name="position"/>
+    </joint>
+    <joint name="yq3_Joint">
+      <command_interface name="position">
+        <param name="min">-1.57</param>
+        <param name="max">1.57</param>
+      </command_interface>
+      <state_interface name="position"/>
+    </joint>
+    <!-- yz - mid left -->
+    <joint name="yz1_Joint">
+      <command_interface name="position">
+        <param name="min">-1.57</param>
+        <param name="max">1.57</param>
+      </command_interface>
+      <state_interface name="position"/>
+    </joint>
+    <joint name="yz2_Joint">
+      <command_interface name="position">
+        <param name="min">-1.57</param>
+        <param name="max">1.57</param>
+      </command_interface>
+      <state_interface name="position"/>
+    </joint>
+    <joint name="yz3_Joint">
+      <command_interface name="position">
+        <param name="min">-1.57</param>
+        <param name="max">1.57</param>
+      </command_interface>
+      <state_interface name="position"/>
+    </joint>
+    <!-- yh - rear left -->
+    <joint name="yh1_Joint">
+      <command_interface name="position">
+        <param name="min">-1.57</param>
+        <param name="max">1.57</param>
+      </command_interface>
+      <state_interface name="position"/>
+    </joint>
+    <joint name="yh2_Joint">
+      <command_interface name="position">
+        <param name="min">-1.57</param>
+        <param name="max">1.57</param>
+      </command_interface>
+      <state_interface name="position"/>
+    </joint>
+    <joint name="yh3_Joint">
+      <command_interface name="position">
+        <param name="min">-1.57</param>
+        <param name="max">1.57</param>
+      </command_interface>
+      <state_interface name="position"/>
+    </joint>
+  </ros2_control>
 </robot>

Commit message: fix: update joint effort and velocity limits in Muto URDF configuration

File: muto_ws/src/muto_description/urdf/Muto.urdf (robot description, URDF)
Before this commit: robot yahboomcar, 24 links, 23 joints
Joints:
- joint yh1_Joint: limit lower=-1.57 upper=1.57 effort=2.5 velocity=3.14 -> lower=-1.57 upper=1.57 effort=3.5 velocity=7.0
- joint yh2_Joint: limit lower=-1.57 upper=1.57 effort=2.5 velocity=3.14 -> lower=-1.57 upper=1.57 effort=3.5 velocity=7.0
- joint yh3_Joint: limit lower=-1.57 upper=1.57 effort=2.5 velocity=3.14 -> lower=-1.57 upper=1.57 effort=3.5 velocity=7.0
- joint yq1_Joint: limit lower=-1.57 upper=1.57 effort=2.5 velocity=3.14 -> lower=-1.57 upper=1.57 effort=3.5 velocity=7.0
- joint yq2_Joint: limit lower=-1.57 upper=1.57 effort=2.5 velocity=3.14 -> lower=-1.57 upper=1.57 effort=3.5 velocity=7.0
- joint yq3_Joint: limit lower=-1.57 upper=1.57 effort=2.5 velocity=3.14 -> lower=-1.57 upper=1.57 effort=3.5 velocity=7.0
- joint yz1_Joint: limit lower=-1.57 upper=1.57 effort=2.5 velocity=3.14 -> lower=-1.57 upper=1.57 effort=3.5 velocity=7.0
- joint yz2_Joint: limit lower=-1.57 upper=1.57 effort=2.5 velocity=3.14 -> lower=-1.57 upper=1.57 effort=3.5 velocity=7.0
- joint yz3_Joint: limit lower=-1.57 upper=1.57 effort=2.5 velocity=3.14 -> lower=-1.57 upper=1.57 effort=3.5 velocity=7.0
- joint zh1_Joint: limit lower=-1.57 upper=1.57 effort=2.5 velocity=3.14 -> lower=-1.57 upper=1.57 effort=3.5 velocity=7.0
- joint zh2_Joint: limit lower=-1.57 upper=1.57 effort=2.5 velocity=3.14 -> lower=-1.57 upper=1.57 effort=3.5 velocity=7.0
- joint zh3_Joint: limit lower=-1.57 upper=1.57 effort=2.5 velocity=3.14 -> lower=-1.57 upper=1.57 effort=3.5 velocity=7.0
- joint zq1_Joint: limit lower=-1.57 upper=1.57 effort=2.5 velocity=3.14 -> lower=-1.57 upper=1.57 effort=3.5 velocity=7.0
- joint zq2_Joint: limit lower=-1.57 upper=1.57 effort=2.5 velocity=3.14 -> lower=-1.57 upper=1.57 effort=3.5 velocity=7.0
- joint zq3_Joint: limit lower=-1.57 upper=1.57 effort=2.5 velocity=3.14 -> lower=-1.57 upper=1.57 effort=3.5 velocity=7.0
- joint zz1_Joint: limit lower=-1.57 upper=1.57 effort=2.5 velocity=3.14 -> lower=-1.57 upper=1.57 effort=3.5 velocity=7.0
- joint zz2_Joint: limit lower=-1.57 upper=1.57 effort=2.5 velocity=3.14 -> lower=-1.57 upper=1.57 effort=3.5 velocity=7.0
- joint zz3_Joint: limit lower=-1.57 upper=1.57 effort=2.5 velocity=3.14 -> lower=-1.57 upper=1.57 effort=3.5 velocity=7.0

Commit message: fix: update joint effort limits in Muto URDF configuration

File: muto_ws/src/muto_description/urdf/Muto.urdf (robot description, URDF)
Before this commit: robot yahboomcar, 24 links, 23 joints
Joints:
- joint yh1_Joint: limit lower=-1.57 upper=1.57 effort=3.5 velocity=7.0 -> lower=-1.57 upper=1.57 effort=4.2 velocity=7.0
- joint yh2_Joint: limit lower=-1.57 upper=1.57 effort=3.5 velocity=7.0 -> lower=-1.57 upper=1.57 effort=4.2 velocity=7.0
- joint yh3_Joint: limit lower=-1.57 upper=1.57 effort=3.5 velocity=7.0 -> lower=-1.57 upper=1.57 effort=4.2 velocity=7.0
- joint yq1_Joint: limit lower=-1.57 upper=1.57 effort=3.5 velocity=7.0 -> lower=-1.57 upper=1.57 effort=4.2 velocity=7.0
- joint yq2_Joint: limit lower=-1.57 upper=1.57 effort=3.5 velocity=7.0 -> lower=-1.57 upper=1.57 effort=4.2 velocity=7.0
- joint yq3_Joint: limit lower=-1.57 upper=1.57 effort=3.5 velocity=7.0 -> lower=-1.57 upper=1.57 effort=4.2 velocity=7.0
- joint yz1_Joint: limit lower=-1.57 upper=1.57 effort=3.5 velocity=7.0 -> lower=-1.57 upper=1.57 effort=4.2 velocity=7.0
- joint yz2_Joint: limit lower=-1.57 upper=1.57 effort=3.5 velocity=7.0 -> lower=-1.57 upper=1.57 effort=4.2 velocity=7.0
- joint yz3_Joint: limit lower=-1.57 upper=1.57 effort=3.5 velocity=7.0 -> lower=-1.57 upper=1.57 effort=4.2 velocity=7.0
- joint zh1_Joint: limit lower=-1.57 upper=1.57 effort=3.5 velocity=7.0 -> lower=-1.57 upper=1.57 effort=4.2 velocity=7.0
- joint zh2_Joint: limit lower=-1.57 upper=1.57 effort=3.5 velocity=7.0 -> lower=-1.57 upper=1.57 effort=4.2 velocity=7.0
- joint zh3_Joint: limit lower=-1.57 upper=1.57 effort=3.5 velocity=7.0 -> lower=-1.57 upper=1.57 effort=4.2 velocity=7.0
- joint zq1_Joint: limit lower=-1.57 upper=1.57 effort=3.5 velocity=7.0 -> lower=-1.57 upper=1.57 effort=4.2 velocity=7.0
- joint zq2_Joint: limit lower=-1.57 upper=1.57 effort=3.5 velocity=7.0 -> lower=-1.57 upper=1.57 effort=4.2 velocity=7.0
- joint zq3_Joint: limit lower=-1.57 upper=1.57 effort=3.5 velocity=7.0 -> lower=-1.57 upper=1.57 effort=4.2 velocity=7.0
- joint zz1_Joint: limit lower=-1.57 upper=1.57 effort=3.5 velocity=7.0 -> lower=-1.57 upper=1.57 effort=4.2 velocity=7.0
- joint zz2_Joint: limit lower=-1.57 upper=1.57 effort=3.5 velocity=7.0 -> lower=-1.57 upper=1.57 effort=4.2 velocity=7.0
- joint zz3_Joint: limit lower=-1.57 upper=1.57 effort=3.5 velocity=7.0 -> lower=-1.57 upper=1.57 effort=4.2 velocity=7.0

Commit message: Refactor code structure for improved readability and maintainability

File: muto_ws/src/muto_description/urdf/Muto.urdf (robot description, URDF)
Before this commit: robot yahboomcar, 24 links, 23 joints
Joints:
- joint yh1_Joint: limit lower=-1.57 upper=1.57 effort=4.2 velocity=7.0 -> lower=-1.3 upper=1.3 effort=4.2 velocity=7.0
- joint yh3_Joint: limit lower=-1.57 upper=1.57 effort=4.2 velocity=7.0 -> lower=-1.57 upper=0.8 effort=4.2 velocity=7.0
- joint yq1_Joint: limit lower=-1.57 upper=1.57 effort=4.2 velocity=7.0 -> lower=-1.3 upper=1.3 effort=4.2 velocity=7.0
- joint yq3_Joint: limit lower=-1.57 upper=1.57 effort=4.2 velocity=7.0 -> lower=-1.57 upper=0.8 effort=4.2 velocity=7.0
- joint yz1_Joint: limit lower=-1.57 upper=1.57 effort=4.2 velocity=7.0 -> lower=-1.3 upper=1.3 effort=4.2 velocity=7.0
- joint yz3_Joint: limit lower=-1.57 upper=1.57 effort=4.2 velocity=7.0 -> lower=-1.57 upper=0.8 effort=4.2 velocity=7.0
- joint zh1_Joint: limit lower=-1.57 upper=1.57 effort=4.2 velocity=7.0 -> lower=-1.3 upper=1.3 effort=4.2 velocity=7.0
- joint zh3_Joint: limit lower=-1.57 upper=1.57 effort=4.2 velocity=7.0 -> lower=-1.57 upper=0.8 effort=4.2 velocity=7.0
- joint zq1_Joint: limit lower=-1.57 upper=1.57 effort=4.2 velocity=7.0 -> lower=-1.3 upper=1.3 effort=4.2 velocity=7.0
- joint zq3_Joint: limit lower=-1.57 upper=1.57 effort=4.2 velocity=7.0 -> lower=-1.57 upper=0.8 effort=4.2 velocity=7.0
- joint zz1_Joint: limit lower=-1.57 upper=1.57 effort=4.2 velocity=7.0 -> lower=-1.3 upper=1.3 effort=4.2 velocity=7.0
- joint zz3_Joint: limit lower=-1.57 upper=1.57 effort=4.2 velocity=7.0 -> lower=-1.57 upper=0.8 effort=4.2 velocity=7.0

File: muto_ws/src/muto_description/urdf/Muto_2.urdf (robot description, URDF)
Before this commit: robot yahboomcar, 24 links, 23 joints
Joints:
- joint yh1_Joint: limit lower=-1.57 upper=1.57 effort=4.2 velocity=7.0 -> lower=-1.3 upper=1.3 effort=4.2 velocity=7.0
- joint yh3_Joint: limit lower=-1.57 upper=1.57 effort=4.2 velocity=7.0 -> lower=-1.57 upper=0.8 effort=4.2 velocity=7.0
- joint yq1_Joint: limit lower=-1.57 upper=1.57 effort=4.2 velocity=7.0 -> lower=-1.3 upper=1.3 effort=4.2 velocity=7.0
- joint yq3_Joint: limit lower=-1.57 upper=1.57 effort=4.2 velocity=7.0 -> lower=-1.57 upper=0.8 effort=4.2 velocity=7.0
- joint yz1_Joint: limit lower=-1.57 upper=1.57 effort=4.2 velocity=7.0 -> lower=-1.3 upper=1.3 effort=4.2 velocity=7.0
- joint yz3_Joint: limit lower=-1.57 upper=1.57 effort=4.2 velocity=7.0 -> lower=-1.57 upper=0.8 effort=4.2 velocity=7.0
- joint zh1_Joint: limit lower=-1.57 upper=1.57 effort=4.2 velocity=7.0 -> lower=-1.3 upper=1.3 effort=4.2 velocity=7.0
- joint zh3_Joint: limit lower=-1.57 upper=1.57 effort=4.2 velocity=7.0 -> lower=-1.57 upper=0.8 effort=4.2 velocity=7.0
- joint zq1_Joint: limit lower=-1.57 upper=1.57 effort=4.2 velocity=7.0 -> lower=-1.3 upper=1.3 effort=4.2 velocity=7.0
- joint zq3_Joint: limit lower=-1.57 upper=1.57 effort=4.2 velocity=7.0 -> lower=-1.57 upper=0.8 effort=4.2 velocity=7.0
- joint zz1_Joint: limit lower=-1.57 upper=1.57 effort=4.2 velocity=7.0 -> lower=-1.3 upper=1.3 effort=4.2 velocity=7.0
- joint zz3_Joint: limit lower=-1.57 upper=1.57 effort=4.2 velocity=7.0 -> lower=-1.57 upper=0.8 effort=4.2 velocity=7.0

Commit message: feat: Fix joint origin and naming issues in URDF due to SolidWorks export bugs

File: muto_ws/src/muto_description/urdf/Muto.urdf (robot description, URDF)
Before this commit: robot yahboomcar, 24 links, 23 joints
Joints:
- joint yz3_Joint: origin xyz=0.195684337632199 -0.0250512362876254 0.015861531236519 rpy=0 0 0 -> xyz=0.0497740601308618 -0.0250512362876254 0.015861531236519 rpy=0 0 0

File: muto_ws/src/muto_description/urdf/Muto_2.urdf (robot description, URDF)
Before this commit: robot yahboomcar, 24 links, 23 joints
Joints:
- joint yz3_Joint: origin xyz=0.195684337632199 -0.0250512362876254 0.015861531236519 rpy=0 0 0 -> xyz=0.0497740601308618 -0.0250512362876254 0.015861531236519 rpy=0 0 0

Commit message: feat: Correct yz3_Link and yz3_Joint parameters for symmetry with zz3_Link

File: muto_ws/src/muto_description/urdf/Muto.urdf (robot description, URDF)
Before this commit: robot yahboomcar, 24 links, 23 joints
Links:
- link yz3_Link: mass 0.0295670684923118 -> 0.0280435236825223
Joints:
- joint yz3_Joint: axis 0.711636313809377 0.702548045949743 0 -> 1 0 0; origin xyz=0.0497740601308618 -0.0250512362876254 0.015861531236519 rpy=0 0 0 -> xyz=0 -0.0708479091470208 0.0158615312365403 rpy=0 0 0

File: muto_ws/src/muto_description/urdf/Muto_2.urdf (robot description, URDF)
Before this commit: robot yahboomcar, 24 links, 23 joints
Links:
- link yz3_Link: mass 0.0295670684923118 -> 0.0280435236825223
Joints:
- joint yz3_Joint: axis 0.711636313809377 0.702548045949743 0 -> 1 0 0; origin xyz=0.0497740601308618 -0.0250512362876254 0.015861531236519 rpy=0 0 0 -> xyz=0 -0.0708479091470208 0.0158615312365403 rpy=0 0 0

Commit message: Refactor URDF files and update gazebo integration
- Updated Muto.urdf with new links and joints for improved symmetry and corrected naming conventions.
- Removed obsolete Muto_2.urdf file to streamline the project structure.
- Modified Muto_gazebo.urdf.xacro to include the updated Muto.urdf instead of the deprecated Muto_2.urdf.

File: muto_ws/src/muto_description/urdf/Muto.urdf (robot description, URDF)
Before this commit: robot yahboomcar, 24 links, 23 joints
Joints:
- removed joint imu_link
- added joint imu_joint: type fixed, parent base_link, child imu_link, origin xyz=0.050316 0.0047788 0.053291 rpy=0 0 0, axis 0 0 0

File: muto_ws/src/muto_description/urdf/Muto_gazebo.urdf.xacro (robot description, xacro)
@@ -7,5 +7,5 @@
     <origin xyz="0 0 0" rpy="0 0 0"/>
   </joint>
-  <xacro:include filename="$(find muto_description)/urdf/Muto_2.urdf"/>
+  <xacro:include filename="$(find muto_description)/urdf/Muto.urdf"/>
   <ros2_control name="MutoHardwareInterface" type="system">
     <hardware>

Commit message: feat: Update yz3_Link and joint parameters for improved symmetry and fix inertia values

File: muto_ws/src/muto_description/urdf/Muto.urdf (robot description, URDF)
Before this commit: robot yahboomcar, 24 links, 23 joints
Joints:
- removed joint imu_joint
- added joint imu_link: type fixed, parent base_link, child imu_link, origin xyz=0.050316 0.0047788 0.053291 rpy=0 0 0, axis 0 0 0
