Commit message: Implement code changes to enhance functionality and improve performance

File: muto_ws/src/muto_description/urdf/Muto.urdf (robot description, URDF)
Before this commit: robot yahboomcar, 24 links, 23 joints
Joints:
- joint yh1_Joint: limit lower=-1.3 upper=1.3 effort=4.2 velocity=7.0 -> lower=-1.57 upper=1.57 effort=4.2 velocity=7.0
- joint yh3_Joint: limit lower=-1.57 upper=0.8 effort=4.2 velocity=7.0 -> lower=-1.57 upper=1.57 effort=4.2 velocity=7.0
- joint yq1_Joint: limit lower=-1.3 upper=1.3 effort=4.2 velocity=7.0 -> lower=-1.57 upper=1.57 effort=4.2 velocity=7.0
- joint yq3_Joint: limit lower=-1.57 upper=0.8 effort=4.2 velocity=7.0 -> lower=-1.57 upper=1.57 effort=4.2 velocity=7.0
- joint yz1_Joint: limit lower=-1.3 upper=1.3 effort=4.2 velocity=7.0 -> lower=-1.57 upper=1.57 effort=4.2 velocity=7.0
- joint yz3_Joint: limit lower=-1.57 upper=0.8 effort=4.2 velocity=7.0 -> lower=-1.57 upper=1.57 effort=4.2 velocity=7.0
- joint zh1_Joint: limit lower=-1.3 upper=1.3 effort=4.2 velocity=7.0 -> lower=-1.57 upper=1.57 effort=4.2 velocity=7.0
- joint zh3_Joint: limit lower=-1.57 upper=0.8 effort=4.2 velocity=7.0 -> lower=-1.57 upper=1.57 effort=4.2 velocity=7.0
- joint zq1_Joint: limit lower=-1.3 upper=1.3 effort=4.2 velocity=7.0 -> lower=-1.57 upper=1.57 effort=4.2 velocity=7.0
- joint zq3_Joint: limit lower=-1.57 upper=0.8 effort=4.2 velocity=7.0 -> lower=-1.57 upper=1.57 effort=4.2 velocity=7.0
- joint zz1_Joint: limit lower=-1.3 upper=1.3 effort=4.2 velocity=7.0 -> lower=-1.57 upper=1.57 effort=4.2 velocity=7.0
- joint zz3_Joint: limit lower=-1.57 upper=0.8 effort=4.2 velocity=7.0 -> lower=-1.57 upper=1.57 effort=4.2 velocity=7.0

Commit message: feat: Update yz3_Link and yz3_Joint parameters for improved positioning and inertia values

File: muto_ws/src/muto_description/urdf/Muto.urdf (robot description, URDF)
Before this commit: robot yahboomcar, 24 links, 23 joints
Links:
- link yz3_Link: mass 0.0280435236825223 -> 0.0295670684923118
Joints:
- removed joint imu_link
- added joint imu_joint: type fixed, parent base_link, child imu_link, origin xyz=0.050316 0.0047788 0.053291 rpy=0 0 0, axis 0 0 0
- joint yz3_Joint: axis 1 0 0 -> 0.711636313809377 0.702548045949743 0; origin xyz=0 -0.0708479091470208 0.0158615312365403 rpy=0 0 0 -> xyz=0.195684337632199 -0.0250512362876254 0.015861531236519 rpy=0 0 0

Commit message: feat: Adjust joint limits for improved range of motion and stability

File: muto_ws/src/muto_description/urdf/Muto.urdf (robot description, URDF)
Before this commit: robot yahboomcar, 24 links, 23 joints
Joints:
- joint yh1_Joint: limit lower=-1.57 upper=1.57 effort=4.2 velocity=7.0 -> lower=-1.2 upper=1.2 effort=4.2 velocity=7.0
- joint yh3_Joint: limit lower=-1.57 upper=1.57 effort=4.2 velocity=7.0 -> lower=-1.57 upper=0.7 effort=4.2 velocity=7.0
- joint yq1_Joint: limit lower=-1.57 upper=1.57 effort=4.2 velocity=7.0 -> lower=-1.2 upper=1.2 effort=4.2 velocity=7.0
- joint yq3_Joint: limit lower=-1.57 upper=1.57 effort=4.2 velocity=7.0 -> lower=-1.57 upper=0.7 effort=4.2 velocity=7.0
- joint yz1_Joint: limit lower=-1.57 upper=1.57 effort=4.2 velocity=7.0 -> lower=-1.2 upper=1.2 effort=4.2 velocity=7.0
- joint yz3_Joint: limit lower=-1.57 upper=1.57 effort=4.2 velocity=7.0 -> lower=-1.57 upper=0.7 effort=4.2 velocity=7.0
- joint zh1_Joint: limit lower=-1.57 upper=1.57 effort=4.2 velocity=7.0 -> lower=-1.2 upper=1.2 effort=4.2 velocity=7.0
- joint zh3_Joint: limit lower=-1.57 upper=1.57 effort=4.2 velocity=7.0 -> lower=-1.57 upper=0.7 effort=4.2 velocity=7.0
- joint zq1_Joint: limit lower=-1.57 upper=1.57 effort=4.2 velocity=7.0 -> lower=-1.2 upper=1.2 effort=4.2 velocity=7.0
- joint zq3_Joint: limit lower=-1.57 upper=1.57 effort=4.2 velocity=7.0 -> lower=-1.57 upper=0.7 effort=4.2 velocity=7.0
- joint zz1_Joint: limit lower=-1.57 upper=1.57 effort=4.2 velocity=7.0 -> lower=-1.2 upper=1.2 effort=4.2 velocity=7.0
- joint zz3_Joint: limit lower=-1.57 upper=1.57 effort=4.2 velocity=7.0 -> lower=-1.57 upper=0.7 effort=4.2 velocity=7.0

Commit message: Implement code changes to enhance functionality and improve performance

File: muto_ws/src/muto_description/urdf/Muto.urdf (robot description, URDF)
Before this commit: robot yahboomcar, 24 links, 23 joints
Joints:
- joint yz3_Joint: origin xyz=0.195684337632199 -0.0250512362876254 0.015861531236519 rpy=0 0 0 -> xyz=0 -0.0708479091470208 0.0158615312365403 rpy=0 0 0

Commit message: Implement code changes to enhance functionality and improve performance

File: muto_ws/src/muto_description/urdf/Muto.urdf (robot description, URDF)
Before this commit: robot yahboomcar, 24 links, 23 joints
Joints:
- joint yz3_Joint: origin xyz=0 -0.0708479091470208 0.0158615312365403 rpy=0 0 0 -> xyz=0.195684337632199 -0.0250512362876254 0.015861531236519 rpy=0 0 0

Commit message: Implement feature X to enhance user experience and optimize performance

File: muto_ws/src/muto_description/urdf/Muto.urdf (robot description, URDF)
Before this commit: robot muto_robot, 24 links, 23 joints
Links:
- removed link laser_scan_fix
- link base_link: geometry collision mesh filename=package://yahboomcar_description/meshes/base_link.STL; visual mesh filename=package://yahboomcar_description/meshes/base_link.STL
- link camera_link: geometry collision mesh filename=package://yahboomcar_description/meshes/camera_Link.STL; visual mesh filename=package://yahboomcar_description/meshes/camera_Link.STL
- link imu_link: geometry collision mesh filename=package://yahboomcar_description/meshes/imu_Link.STL; visual mesh filename=package://yahboomcar_description/meshes/imu_Link.STL
- link laser: geometry collision mesh filename=package://yahboomcar_description/meshes/LD_Link.STL; visual mesh filename=package://yahboomcar_description/meshes/LD_Link.STL
- link yh1_Link: geometry collision mesh filename=package://yahboomcar_description/meshes/yh1_Link.STL; visual mesh filename=package://yahboomcar_description/meshes/yh1_Link.STL
- link yh2_Link: geometry collision mesh filename=package://yahboomcar_description/meshes/yh2_Link.STL; visual mesh filename=package://yahboomcar_description/meshes/yh2_Link.STL
- link yh3_Link: geometry collision mesh filename=package://yahboomcar_description/meshes/yh3_Link.STL; visual mesh filename=package://yahboomcar_description/meshes/yh3_Link.STL
- link yq1_Link: geometry collision mesh filename=package://yahboomcar_description/meshes/yq1_Link.STL; visual mesh filename=package://yahboomcar_description/meshes/yq1_Link.STL
- link yq2_Link: geometry collision mesh filename=package://yahboomcar_description/meshes/yq2_Link.STL; visual mesh filename=package://yahboomcar_description/meshes/yq2_Link.STL
- link yq3_Link: geometry collision mesh filename=package://yahboomcar_description/meshes/yq3_Link.STL; visual mesh filename=package://yahboomcar_description/meshes/yq3_Link.STL
- link yz1_Link: geometry collision mesh filename=package://yahboomcar_description/meshes/yz1_Link.STL; visual mesh filename=package://yahboomcar_description/meshes/yz1_Link.STL
- link yz2_Link: geometry collision mesh filename=package://yahboomcar_description/meshes/yz2_Link.STL; visual mesh filename=package://yahboomcar_description/meshes/yz2_Link.STL
- link yz3_Link: geometry collision mesh filename=package://yahboomcar_description/meshes/yz3_Link.STL; visual mesh filename=package://yahboomcar_description/meshes/yz3_Link.STL
- link zh1_Link: geometry collision mesh filename=package://yahboomcar_description/meshes/zh1_Link.STL; visual mesh filename=package://yahboomcar_description/meshes/zh1_Link.STL
- link zh2_Link: geometry collision mesh filename=package://yahboomcar_description/meshes/zh2_Link.STL; visual mesh filename=package://yahboomcar_description/meshes/zh2_Link.STL
- link zh3_Link: geometry collision mesh filename=package://yahboomcar_description/meshes/zh3_Link.STL; visual mesh filename=package://yahboomcar_description/meshes/zh3_Link.STL
- link zq1_Link: geometry collision mesh filename=package://yahboomcar_description/meshes/zq1_Link.STL; visual mesh filename=package://yahboomcar_description/meshes/zq1_Link.STL
- link zq2_Link: geometry collision mesh filename=package://yahboomcar_description/meshes/zq2_Link.STL; visual mesh filename=package://yahboomcar_description/meshes/zq2_Link.STL
- link zq3_Link: geometry collision mesh filename=package://yahboomcar_description/meshes/zq3_Link.STL; visual mesh filename=package://yahboomcar_description/meshes/zq3_Link.STL
- link zz1_Link: geometry collision mesh filename=package://yahboomcar_description/meshes/zz1_Link.STL; visual mesh filename=package://yahboomcar_description/meshes/zz1_Link.STL
- link zz2_Link: geometry collision mesh filename=package://yahboomcar_description/meshes/zz2_Link.STL; visual mesh filename=package://yahboomcar_description/meshes/zz2_Link.STL
- link zz3_Link: geometry collision mesh filename=package://yahboomcar_description/meshes/zz3_Link.STL; visual mesh filename=package://yahboomcar_description/meshes/zz3_Link.STL
Joints:
- removed joint laser_scan_fix_joint
- removed joint yh2_Joint
- removed joint yh3_Joint
- added joint yh2_joint: type revolute, parent yh1_Link, child yh2_Link, origin xyz=-0.055226635669978 -0.0165734288280502 -0.027473927115545 rpy=0 0 0, axis -0.711636313809332 0.702548045949788 0, limit lower=-1.57 upper=1.57 effort=0 velocity=0
- added joint yh3_joint: type revolute, parent yh2_Link, child yh3_Link, origin xyz=-0.0497740601308654 -0.0504179449064808 0.0158615312365509 rpy=0 0 0, axis 0.711636313809335 -0.702548045949785 0, limit lower=-1.57 upper=1.57 effort=0 velocity=0
- joint LD_Joint: origin xyz=-0.0316436626639546 0 0.183666853069193 rpy=0 0 0 -> xyz=-0.0316436626639546 0 0.183666853069193 rpy=0 0 3.14
- joint footprint_Joint: child base_footprint -> base_link; origin xyz=0 0 -0.113 rpy=0 0 0 -> xyz=0 0 0.113 rpy=0 0 0; parent base_link -> base_footprint
- joint yh1_Joint: limit lower=-1.2 upper=1.2 effort=4.2 velocity=7.0 -> lower=-1.57 upper=1.57 effort=0 velocity=0
- joint yq1_Joint: limit lower=-1.2 upper=1.2 effort=4.2 velocity=7.0 -> lower=-1.57 upper=1.57 effort=0 velocity=0
- joint yq2_Joint: limit lower=-1.57 upper=1.57 effort=4.2 velocity=7.0 -> lower=-1.57 upper=1.57 effort=0 velocity=0
- joint yq3_Joint: limit lower=-1.57 upper=0.7 effort=4.2 velocity=7.0 -> lower=-1.57 upper=1.57 effort=0 velocity=0
- joint yz1_Joint: limit lower=-1.2 upper=1.2 effort=4.2 velocity=7.0 -> lower=-1.57 upper=1.57 effort=0 velocity=0
- joint yz2_Joint: limit lower=-1.57 upper=1.57 effort=4.2 velocity=7.0 -> lower=-1.57 upper=1.57 effort=0 velocity=0
- joint yz3_Joint: limit lower=-1.57 upper=0.7 effort=4.2 velocity=7.0 -> lower=-1.57 upper=1.57 effort=0 velocity=0; origin xyz=0 -0.0708479091470208 0.0158615312365403 rpy=0 0 0 -> xyz=0.195684337632199 -0.0250512362876254 0.015861531236519 rpy=0 0 0
- joint zh1_Joint: limit lower=-1.2 upper=1.2 effort=4.2 velocity=7.0 -> lower=-1.57 upper=1.57 effort=0 velocity=0
- joint zh2_Joint: limit lower=-1.57 upper=1.57 effort=4.2 velocity=7.0 -> lower=-1.57 upper=1.57 effort=0 velocity=0
- joint zh3_Joint: limit lower=-1.57 upper=0.7 effort=4.2 velocity=7.0 -> lower=-1.57 upper=1.57 effort=0 velocity=0
- joint zq1_Joint: limit lower=-1.2 upper=1.2 effort=4.2 velocity=7.0 -> lower=-1.57 upper=1.57 effort=0 velocity=0
- joint zq2_Joint: limit lower=-1.57 upper=1.57 effort=4.2 velocity=7.0 -> lower=-1.57 upper=1.57 effort=0 velocity=0
- joint zq3_Joint: limit lower=-1.57 upper=0.7 effort=4.2 velocity=7.0 -> lower=-1.57 upper=1.57 effort=0 velocity=0
- joint zz1_Joint: limit lower=-1.2 upper=1.2 effort=4.2 velocity=7.0 -> lower=-1.57 upper=1.57 effort=0 velocity=0
- joint zz2_Joint: limit lower=-1.57 upper=1.57 effort=4.2 velocity=7.0 -> lower=-1.57 upper=1.57 effort=0 velocity=0
- joint zz3_Joint: limit lower=-1.57 upper=0.7 effort=4.2 velocity=7.0 -> lower=-1.57 upper=1.57 effort=0 velocity=0

Commit message: feat: Update Muto URDF to reference new mesh file paths and remove obsolete USD configuration files

File: muto_ws/src/muto_description/urdf/Muto.urdf (robot description, URDF)
Before this commit: robot yahboomcar, 23 links, 22 joints
Links:
- link base_link: geometry collision mesh filename=package://muto_description/meshes/base_link.STL; visual mesh filename=package://muto_description/meshes/base_link.STL
- link camera_link: geometry collision mesh filename=package://muto_description/meshes/camera_Link.STL; visual mesh filename=package://muto_description/meshes/camera_Link.STL
- link imu_link: geometry collision mesh filename=package://muto_description/meshes/imu_Link.STL; visual mesh filename=package://muto_description/meshes/imu_Link.STL
- link laser: geometry collision mesh filename=package://muto_description/meshes/LD_Link.STL; visual mesh filename=package://muto_description/meshes/LD_Link.STL
- link yh1_Link: geometry collision mesh filename=package://muto_description/meshes/yh1_Link.STL; visual mesh filename=package://muto_description/meshes/yh1_Link.STL
- link yh2_Link: geometry collision mesh filename=package://muto_description/meshes/yh2_Link.STL; visual mesh filename=package://muto_description/meshes/yh2_Link.STL
- link yh3_Link: geometry collision mesh filename=package://muto_description/meshes/yh3_Link.STL; visual mesh filename=package://muto_description/meshes/yh3_Link.STL
- link yq1_Link: geometry collision mesh filename=package://muto_description/meshes/yq1_Link.STL; visual mesh filename=package://muto_description/meshes/yq1_Link.STL
- link yq2_Link: geometry collision mesh filename=package://muto_description/meshes/yq2_Link.STL; visual mesh filename=package://muto_description/meshes/yq2_Link.STL
- link yq3_Link: geometry collision mesh filename=package://muto_description/meshes/yq3_Link.STL; visual mesh filename=package://muto_description/meshes/yq3_Link.STL
- link yz1_Link: geometry collision mesh filename=package://muto_description/meshes/yz1_Link.STL; visual mesh filename=package://muto_description/meshes/yz1_Link.STL
- link yz2_Link: geometry collision mesh filename=package://muto_description/meshes/yz2_Link.STL; visual mesh filename=package://muto_description/meshes/yz2_Link.STL
- link yz3_Link: geometry collision mesh filename=package://muto_description/meshes/yz3_Link.STL; visual mesh filename=package://muto_description/meshes/yz3_Link.STL
- link zh1_Link: geometry collision mesh filename=package://muto_description/meshes/zh1_Link.STL; visual mesh filename=package://muto_description/meshes/zh1_Link.STL
- link zh2_Link: geometry collision mesh filename=package://muto_description/meshes/zh2_Link.STL; visual mesh filename=package://muto_description/meshes/zh2_Link.STL
- link zh3_Link: geometry collision mesh filename=package://muto_description/meshes/zh3_Link.STL; visual mesh filename=package://muto_description/meshes/zh3_Link.STL
- link zq1_Link: geometry collision mesh filename=package://muto_description/meshes/zq1_Link.STL; visual mesh filename=package://muto_description/meshes/zq1_Link.STL
- link zq2_Link: geometry collision mesh filename=package://muto_description/meshes/zq2_Link.STL; visual mesh filename=package://muto_description/meshes/zq2_Link.STL
- link zq3_Link: geometry collision mesh filename=package://muto_description/meshes/zq3_Link.STL; visual mesh filename=package://muto_description/meshes/zq3_Link.STL
- link zz1_Link: geometry collision mesh filename=package://muto_description/meshes/zz1_Link.STL; visual mesh filename=package://muto_description/meshes/zz1_Link.STL
- link zz2_Link: geometry collision mesh filename=package://muto_description/meshes/zz2_Link.STL; visual mesh filename=package://muto_description/meshes/zz2_Link.STL
- link zz3_Link: geometry collision mesh filename=package://muto_description/meshes/zz3_Link.STL; visual mesh filename=package://muto_description/meshes/zz3_Link.STL
