Commit message: Implement feature X to enhance user experience and optimize performance

File: muto_ws/src/muto_description/urdf/Muto.urdf (robot description, URDF)
Before this commit: robot yahboomcar, 23 links, 22 joints
Links:
- removed link base_footprint
- removed link base_link
- removed link camera_link
- removed link imu_link
- removed link laser
- removed link yh1_Link
- removed link yh2_Link
- removed link yh3_Link
- removed link yq1_Link
- removed link yq2_Link
- removed link yq3_Link
- removed link yz1_Link
- removed link yz2_Link
- removed link yz3_Link
- removed link zh1_Link
- removed link zh2_Link
- removed link zh3_Link
- removed link zq1_Link
- removed link zq2_Link
- removed link zq3_Link
- removed link zz1_Link
- removed link zz2_Link
- removed link zz3_Link
- added link robot1/base_footprint
- added link robot1/base_link, mass 0.53214037432126; collision mesh filename=package://muto_description/meshes/base_link.STL; visual mesh filename=package://muto_description/meshes/base_link.STL
- added link robot1/camera_link, mass 0.224644099483613; collision mesh filename=package://muto_description/meshes/camera_Link.STL; visual mesh filename=package://muto_description/meshes/camera_Link.STL
- added link robot1/imu_link, mass 0.0109726593021096; collision mesh filename=package://muto_description/meshes/IMU_Link.STL; visual mesh filename=package://muto_description/meshes/IMU_Link.STL
- added link robot1/laser, mass 0.0512442437357772; collision mesh filename=package://muto_description/meshes/Lider_Link.STL; visual mesh filename=package://muto_description/meshes/Lider_Link.STL
- added link robot1/yh1_Link, mass 0.00573728308905327; collision mesh filename=package://muto_description/meshes/yh1_Link.STL; visual mesh filename=package://muto_description/meshes/yh1_Link.STL
- added link robot1/yh2_Link, mass 0.0134955335598432; collision mesh filename=package://muto_description/meshes/yh2_Link.STL; visual mesh filename=package://muto_description/meshes/yh2_Link.STL
- added link robot1/yh3_Link, mass 0.0186861004150177; collision mesh filename=package://muto_description/meshes/yh3_Link.STL; visual mesh filename=package://muto_description/meshes/yh3_Link.STL
- added link robot1/yq1_Link, mass 0.00573728308905327; collision mesh filename=package://muto_description/meshes/yq1_Link.STL; visual mesh filename=package://muto_description/meshes/yq1_Link.STL
- added link robot1/yq2_Link, mass 0.0134955335011356; collision mesh filename=package://muto_description/meshes/yq2_Link.STL; visual mesh filename=package://muto_description/meshes/yq2_Link.STL
- added link robot1/yq3_Link, mass 0.0186861004150177; collision mesh filename=package://muto_description/meshes/yq3_Link.STL; visual mesh filename=package://muto_description/meshes/yq3_Link.STL
- added link robot1/yz1_Link, mass 0.00573728308905327; collision mesh filename=package://muto_description/meshes/yz1_Link.STL; visual mesh filename=package://muto_description/meshes/yz1_Link.STL
- added link robot1/yz2_Link, mass 0.0134955337243651; collision mesh filename=package://muto_description/meshes/yz2_Link.STL; visual mesh filename=package://muto_description/meshes/yz2_Link.STL
- added link robot1/yz3_Link, mass 0.0186861004150178; collision mesh filename=package://muto_description/meshes/yz3_Link.STL; visual mesh filename=package://muto_description/meshes/yz3_Link.STL
- added link robot1/zh1_Link, mass 0.00573728308905326; collision mesh filename=package://muto_description/meshes/zh1_Link.STL; visual mesh filename=package://muto_description/meshes/zh1_Link.STL
- added link robot1/zh2_Link, mass 0.0134955335748432; collision mesh filename=package://muto_description/meshes/zh2_Link.STL; visual mesh filename=package://muto_description/meshes/zh2_Link.STL
- added link robot1/zh3_Link, mass 0.0186861004150177; collision mesh filename=package://muto_description/meshes/zh3_Link.STL; visual mesh filename=package://muto_description/meshes/zh3_Link.STL
- added link robot1/zq1_Link, mass 0.00573728308905327; collision mesh filename=package://muto_description/meshes/zq1_Link.STL; visual mesh filename=package://muto_description/meshes/zq1_Link.STL
- added link robot1/zq2_Link, mass 0.0134955335282745; collision mesh filename=package://muto_description/meshes/zq2_Link.STL; visual mesh filename=package://muto_description/meshes/zq2_Link.STL
- added link robot1/zq3_Link, mass 0.0186861004150177; collision mesh filename=package://muto_description/meshes/zq3_Link.STL; visual mesh filename=package://muto_description/meshes/zq3_Link.STL
- added link robot1/zz1_Link, mass 0.00573728308905326; collision mesh filename=package://muto_description/meshes/zz1_Link.STL; visual mesh filename=package://muto_description/meshes/zz1_Link.STL
- added link robot1/zz2_Link, mass 0.013495533786557; collision mesh filename=package://muto_description/meshes/zz2_Link.STL; visual mesh filename=package://muto_description/meshes/zz2_Link.STL
- added link robot1/zz3_Link, mass 0.0186861004150177; collision mesh filename=package://muto_description/meshes/zz3_Link.STL; visual mesh filename=package://muto_description/meshes/zz3_Link.STL
Joints:
- removed joint LD_Joint
- removed joint imu_joint
- removed joint yh2_joint
- removed joint yh3_joint
- added joint IMU_Joint: type fixed, parent robot1/base_link, child robot1/imu_link, origin xyz=0.0504496004683106 -0.0053215233667368 0.00919143934 rpy=0 0 0, axis 0 0 0
- added joint Lider_Joint: type fixed, parent robot1/base_link, child robot1/laser, origin xyz=-0.0342026208580557 0 0.131558291660108 rpy=0 0 3.14, axis 0 0 0
- added joint yh2_Joint: type revolute, parent robot1/yh1_Link, child robot1/yh2_Link, origin xyz=-0.0565637048839115 -0.0111895987572697 -0.027473927115545 rpy=0 0 0, axis -0.640829895528474 0.767682906542125 0, limit lower=-1 upper=1 effort=0 velocity=0
- added joint yh3_Joint: type revolute, parent robot1/yh2_Link, child robot1/yh3_Link, origin xyz=-0.0553326362497745 -0.0461893930499636 -0.00870995979721381 rpy=0 0 0, axis 0.640829895528473 -0.767682906542126 0, limit lower=-1 upper=1 effort=0 velocity=0
- joint camera_Joint: child camera_link -> robot1/camera_link; origin xyz=0.070673 0 0.12267 rpy=0 0 0 -> xyz=0.0710921136864663 0 0.095735206628551 rpy=0 0 0; parent base_link -> robot1/base_link
- joint footprint_Joint: child base_link -> robot1/base_link; origin xyz=0 0 0.113 rpy=0 0 0 -> xyz=0 0 0.173564572468554 rpy=0 0 0; parent base_footprint -> robot1/base_footprint
- joint yh1_Joint: child yh1_Link -> robot1/yh1_Link; limit lower=-1.57 upper=1.57 effort=0 velocity=0 -> lower=-1 upper=1 effort=0 velocity=0; origin xyz=-0.10239 -0.050691 0.05005 rpy=0 0 0 -> xyz=-0.102390617184867 -0.0506909842824246 0.00890303231720998 rpy=0 0 0; parent base_link -> robot1/base_link
- joint yq1_Joint: child yq1_Link -> robot1/yq1_Link; limit lower=-1.57 upper=1.57 effort=0 velocity=0 -> lower=-1 upper=1 effort=0 velocity=0; origin xyz=0.10239 -0.050692 0.05005 rpy=0 0 0 -> xyz=0.102389778497169 -0.0506918122592142 0.00890303231680312 rpy=0 0 0; parent base_link -> robot1/base_link
- joint yq2_Joint: axis -0.711636313809368 -0.702548045949752 0 -> -0.650697741083124 -0.759336848670812 0; child yq2_Link -> robot1/yq2_Link; limit lower=-1.57 upper=1.57 effort=0 velocity=0 -> lower=-1 upper=1 effort=0 velocity=0; origin xyz=0.0158622603425983 -0.0554350839033059 -0.027473927115545 rpy=0 0 0 -> xyz=0.0204208290570828 -0.0539226257814318 -0.027473927115545 rpy=0 0 0; parent yq1_Link -> robot1/yq1_Link
- joint yq3_Joint: axis 0.711636313809377 0.702548045949743 0 -> 0.650697741083089 0.759336848670842 0; child yq3_Link -> robot1/yq3_Link; limit lower=-1.57 upper=1.57 effort=0 velocity=0 -> lower=-1 upper=1 effort=0 velocity=0; origin xyz=0.049774060130825 -0.0504179449064464 0.0158615312365191 rpy=0 0 0 -> xyz=0.0545867151865156 -0.0467769374380216 -0.0101603500661879 rpy=0 0 0; parent yq2_Link -> robot1/yq2_Link
- joint yz1_Joint: child yz1_Link -> robot1/yz1_Link; limit lower=-1.57 upper=1.57 effort=0 velocity=0 -> lower=-1 upper=1 effort=0 velocity=0; origin xyz=0 -0.0809 0.05005 rpy=0 0 0 -> xyz=0 -0.0808999860084942 0.00890303231681663 rpy=0 0 0; parent base_link -> robot1/base_link
- joint yz2_Joint: axis -1 0 0 -> -0.999977026444829 0.00677839085316414 0; child yz2_Link -> robot1/yz2_Link; limit lower=-1.57 upper=1.57 effort=0 velocity=0 -> lower=-1 upper=1 effort=0 velocity=0; origin xyz=-0.0276576493944395 -0.0505936187726991 -0.0274739271155447 rpy=0 0 0 -> xyz=-0.0279999573226229 -0.0504049820997311 -0.0274739271155452 rpy=0 0 0; parent yz1_Link -> robot1/yz1_Link
- joint yz3_Joint: axis 0.711636313809377 0.702548045949743 0 -> 0.999977026444829 -0.00677839085317342 0; child yz3_Link -> robot1/yz3_Link; limit lower=-1.57 upper=1.57 effort=0 velocity=0 -> lower=-1 upper=1 effort=0 velocity=0; origin xyz=0.195684337632199 -0.0250512362876254 0.015861531236519 rpy=0 0 0 -> xyz=-0.00048423904144777 -0.0714370014164497 -0.0129438945286439 rpy=0 0 0; parent yz2_Link -> robot1/yz2_Link
- joint zh1_Joint: child zh1_Link -> robot1/zh1_Link; limit lower=-1.57 upper=1.57 effort=0 velocity=0 -> lower=-1 upper=1 effort=0 velocity=0; origin xyz=-0.10239 0.050692 0.05005 rpy=0 0 0 -> xyz=-0.102389778497467 0.0506918122589784 0.00890303231722977 rpy=0 0 0; parent base_link -> robot1/base_link
- joint zh2_Joint: axis 0.711636313809332 0.702548045949789 0 -> 0.718891931205768 0.695121853524432 0; child zh2_Link -> robot1/zh2_Link; limit lower=-1.57 upper=1.57 effort=0 velocity=0 -> lower=-1 upper=1 effort=0 velocity=0; origin xyz=-0.0158622603425981 0.0554350839033061 -0.0274739271155447 rpy=0 0 0 -> xyz=-0.0152858690720031 0.0555967808173864 -0.027473927115545 rpy=0 0 0; parent zh1_Link -> robot1/zh1_Link
- joint zh3_Joint: axis -0.711636313809358 -0.702548045949762 0 -> -0.71889193120591 -0.695121853524285 0; child zh3_Link -> robot1/zh3_Link; limit lower=-1.57 upper=1.57 effort=0 velocity=0 -> lower=-1 upper=1 effort=0 velocity=0; origin xyz=-0.049587285328241 0.0514454617130769 0.0161615312365663 rpy=0 0 0 -> xyz=-0.0498265050927568 0.051530350095747 -0.0115311089514983 rpy=0 0 0; parent zh2_Link -> robot1/zh2_Link
- joint zq1_Joint: child zq1_Link -> robot1/zq1_Link; limit lower=-1.57 upper=1.57 effort=0 velocity=0 -> lower=-1 upper=1 effort=0 velocity=0; origin xyz=0.102390617184867 0.050690984282426 0.05005003231721 rpy=0 0 0 -> xyz=0.102390617184868 0.0506909842824243 0.00890303231720998 rpy=0 0 0; parent base_link -> robot1/base_link
- joint zq2_Joint: axis 0.71164 -0.70255 0 -> 0.817656990289366 -0.575705694110224 0; child zq2_Link -> robot1/zq2_Link; limit lower=-1.57 upper=1.57 effort=0 velocity=0 -> lower=-1 upper=1 effort=0 velocity=0; origin xyz=0.055227 0.016573 -0.027474 rpy=0 0 0 -> xyz=0.0554554222234711 0.015791009358476 -0.0274739271155451 rpy=0 0 0; parent zq1_Link -> robot1/zq1_Link
- joint zq3_Joint: axis -0.711636313809335 0.702548045949785 0 -> -0.701632964361134 0.712538548656708 0; child zq3_Link -> robot1/zq3_Link; limit lower=-1.57 upper=1.57 effort=0 velocity=0 -> lower=-1 upper=1 effort=0 velocity=0; origin xyz=0.0497740601308618 0.0504179449064641 0.0158615312364907 rpy=0 0 0 -> xyz=0.051296151611705 0.0505110509227498 -0.00940013983432441 rpy=0 0 0; parent zq2_Link -> robot1/zq2_Link
- joint zz1_Joint: child zz1_Link -> robot1/zz1_Link; limit lower=-1.57 upper=1.57 effort=0 velocity=0 -> lower=-1 upper=1 effort=0 velocity=0; origin xyz=0 0.0809 0.05005 rpy=0 0 0 -> xyz=0 0.0808999860084089 0.00890303231720998 rpy=0 0 0; parent base_link -> robot1/base_link
- joint zz2_Joint: axis 1 0 0 -> 0.999865151407349 -0.0164219061365844 0; child zz2_Link -> robot1/zz2_Link; limit lower=-1.57 upper=1.57 effort=0 velocity=0 -> lower=-1 upper=1 effort=0 velocity=0; origin xyz=0.0276576493944395 0.0505936187726988 -0.0274739271155451 rpy=0 0 0 -> xyz=0.0284847634579382 0.0501326049720961 -0.027473927115545 rpy=0 0 0; parent zz1_Link -> robot1/zz1_Link
- joint zz3_Joint: axis -1 0 0 -> -0.999865151407349 0.016421906136588 0; child zz3_Link -> robot1/zz3_Link; limit lower=-1.57 upper=1.57 effort=0 velocity=0 -> lower=-1 upper=1 effort=0 velocity=0; origin xyz=0 0.0708479091470208 0.0158615312365403 rpy=0 0 0 -> xyz=0.00117132789043703 0.0713175394365218 -0.0135447637147809 rpy=0 0 0; parent zz2_Link -> robot1/zz2_Link
