Commit message: Add URDF model for Yahboom Car robot
- Created a new URDF file for the Yahboom Car robot, defining its structure, links, joints, and physical properties.
- Included detailed inertial, visual, and collision properties for each link.
- Configured revolute joints with specified limits and axes for movement.
- Integrated meshes for visual representation sourced from the yahboomcar_description package.

File: muto_ws/src/muto_description/urdf/yahboomcar.urdf (robot description, URDF)
Before this commit: robot muto_robot, 24 links, 23 joints
Links:
- link base_link: geometry collision mesh filename=package://yahboomcar_description/meshes/base_link.STL; visual mesh filename=package://yahboomcar_description/meshes/base_link.STL
- link camera_link: geometry collision mesh filename=package://yahboomcar_description/meshes/camera_Link.STL; visual mesh filename=package://yahboomcar_description/meshes/camera_Link.STL
- link imu_link: geometry collision mesh filename=package://yahboomcar_description/meshes/imu_Link.STL; visual mesh filename=package://yahboomcar_description/meshes/imu_Link.STL
- link laser: geometry collision mesh filename=package://yahboomcar_description/meshes/LD_Link.STL; visual mesh filename=package://yahboomcar_description/meshes/LD_Link.STL
- link yh1_Link: geometry collision mesh filename=package://yahboomcar_description/meshes/yh1_Link.STL; visual mesh filename=package://yahboomcar_description/meshes/yh1_Link.STL
- link yh2_Link: geometry collision mesh filename=package://yahboomcar_description/meshes/yh2_Link.STL; visual mesh filename=package://yahboomcar_description/meshes/yh2_Link.STL
- link yh3_Link: geometry collision mesh filename=package://yahboomcar_description/meshes/yh3_Link.STL; visual mesh filename=package://yahboomcar_description/meshes/yh3_Link.STL
- link yq1_Link: geometry collision mesh filename=package://yahboomcar_description/meshes/yq1_Link.STL; visual mesh filename=package://yahboomcar_description/meshes/yq1_Link.STL
- link yq2_Link: geometry collision mesh filename=package://yahboomcar_description/meshes/yq2_Link.STL; visual mesh filename=package://yahboomcar_description/meshes/yq2_Link.STL
- link yq3_Link: geometry collision mesh filename=package://yahboomcar_description/meshes/yq3_Link.STL; visual mesh filename=package://yahboomcar_description/meshes/yq3_Link.STL
- link yz1_Link: geometry collision mesh filename=package://yahboomcar_description/meshes/yz1_Link.STL; visual mesh filename=package://yahboomcar_description/meshes/yz1_Link.STL
- link yz2_Link: geometry collision mesh filename=package://yahboomcar_description/meshes/yz2_Link.STL; visual mesh filename=package://yahboomcar_description/meshes/yz2_Link.STL
- link yz3_Link: geometry collision mesh filename=package://yahboomcar_description/meshes/yz3_Link.STL; visual mesh filename=package://yahboomcar_description/meshes/yz3_Link.STL
- link zh1_Link: geometry collision mesh filename=package://yahboomcar_description/meshes/zh1_Link.STL; visual mesh filename=package://yahboomcar_description/meshes/zh1_Link.STL
- link zh2_Link: geometry collision mesh filename=package://yahboomcar_description/meshes/zh2_Link.STL; visual mesh filename=package://yahboomcar_description/meshes/zh2_Link.STL
- link zh3_Link: geometry collision mesh filename=package://yahboomcar_description/meshes/zh3_Link.STL; visual mesh filename=package://yahboomcar_description/meshes/zh3_Link.STL
- link zq1_Link: geometry collision mesh filename=package://yahboomcar_description/meshes/zq1_Link.STL; visual mesh filename=package://yahboomcar_description/meshes/zq1_Link.STL
- link zq2_Link: geometry collision mesh filename=package://yahboomcar_description/meshes/zq2_Link.STL; visual mesh filename=package://yahboomcar_description/meshes/zq2_Link.STL
- link zq3_Link: geometry collision mesh filename=package://yahboomcar_description/meshes/zq3_Link.STL; visual mesh filename=package://yahboomcar_description/meshes/zq3_Link.STL
- link zz1_Link: geometry collision mesh filename=package://yahboomcar_description/meshes/zz1_Link.STL; visual mesh filename=package://yahboomcar_description/meshes/zz1_Link.STL
- link zz2_Link: geometry collision mesh filename=package://yahboomcar_description/meshes/zz2_Link.STL; visual mesh filename=package://yahboomcar_description/meshes/zz2_Link.STL
- link zz3_Link: geometry collision mesh filename=package://yahboomcar_description/meshes/zz3_Link.STL; visual mesh filename=package://yahboomcar_description/meshes/zz3_Link.STL
